Commit message: fix: align gripper kinematics and accumulate bounded servo targets

File: src/sorter/planning/rmpflow/ur10e.urdf (robot description, URDF)
Before this commit: robot ur_gripper, 15 links, 14 joints
Joints:
- joint ee_link_root_joint: origin xyz=-0. 0. -0.0000001 rpy=0. 0. -1.5707963 -> xyz=-0. 0. -0.0000001 rpy=0. 0. 1.5707963
